File: hw/bluetooth-audio/micro.kicad_sch (KiCad schematic)
At the start: 46 parts, among them J3 Conn_01x06, J4 2x5 JTAG header, Q1 UMH3N, U1 ESP32D0WD-V3, U2 CH340K, U6 W25Q32JVZP, Y1 Crystal 40 MHz 10pF

Commit message: Schematic: split supply into separate audio and system 3V3 rails
First design work since the April 2025 production release. Sixteen months of
edits had accumulated uncommitted; this captures the schematic and board state.

Power topology change: the single 3.3 V supply is now two independent rails,
+3V3_SYS and +3V3_AUDIO, each with its own regulator (U7, U8) and test point
(TEST_3V3_SYS, TEST_3V3_AUDIO). This isolates the ES8388 and the mic from the
~250 mA Bluetooth TX bursts on the ESP32 rail, which design-review-v1 flagged
as an S2 defect and the ES8388 user guide asks for directly.

Also addresses the S1 defects from the review (owner-applied): ES8388 CE pin
pulled down to DGND so the I2C address is determined rather than floating, and
the ESP32 CAP1 10 nF cap fitted.

Both rails are currently NCP1117-3.3 in SOT-223. The topology is right but the
parts are not yet the ones specified in docs/requirements-design.md: Rail A
should become AP7361C-33Y5 (SOT-89-5, ultra-low dropout, needed so the rail
survives on battery) and Rail B an LP5907MFX-3.3 (6.5 uVRMS, the point of
having a separate analog rail at all). Two SOT-223 parts also spend board area
the review specifically asked to reclaim.

Co-Authored-By: Claude Opus 5 <noreply@anthropic.com>
Parts:
- added C45: 10nF, Capacitor_SMD:C_0402_1005Metric, symbol Device:C_Small
Connections:
- net GND: now also C45.1
- net at U1.48 (CAP1): now also C45.2
- no-connect marks 15 -> 14
Other:
- note added: "Check swapped IO2 and IO3"

Commit message: Rev B micro sheet: correctness fixes, CH340 load switch, full ESP32 GPIO map
Micro-sheet fixes (netlist-verified):
- UART TX/RX crossover corrected (U0RXD<->CH340 TXD, U0TXD<->CH340 RXD)
- Flash IO2/IO3 uncrossed (GPIO9/SPIWP->IO2, GPIO10/SPIHD->IO3)
- Digital rail unified to +3V3_SYS; EN pull-up (R11) reconnected

CH340K high-side load switch (delta #16):
- Q2 AO3401A (SOT-23, LCSC C15127) + R40 100k gate pull-down = default-ON
  so the ROM bootloader is powered for USB flashing; gate CH340_EN on GPIO21,
  firmware drives high to disable the bridge on battery

Full ESP32 interface wired (see design-overview.md 3.8):
- EN1->16, EN2->17, AUDIO_VCC_EN->4, AUDIO_SW->5, CH340_EN->21, CHARGE_EN->2
- /PGOOD->38, /CHG->32; ADC1 senses BAT_ADC->34, USB_CC1->36, USB_CC2->37,
  USB_VBUS_SENSE->39; GPIO33 spare
- AUDIO_SW drives both TS5A23159 inputs (LOW=RX, HIGH=TX); pinout verified
  against TI datasheet (COM=jack, NC=codec-out, NO=codec-in, both channels)

Docs:
- design-overview.md: committed GPIO map with strapping-pin FW/HW implications
  (3.8), AUDIO_SW/CHARGE_EN firmware notes (9), updated status (10)
- design-review-micro.md: micro-sheet systems review
- added WCH CH340 datasheet; updated TODO
- gitignore MCP snapshot/log artifacts

Co-Authored-By: Claude Opus 4.8 <noreply@anthropic.com>
Parts:
- added Q2: AO3401A, Package_TO_SOT_SMD:SOT-23, symbol Transistor_FET:AO3401A
- added R40: 100k, Resistor_SMD:R_0402_1005Metric, symbol Device:R
- R12, R18: value 1k -> 330R
Connections:
- net GND: now also R40.2
- net GPIO_2: no longer U1.22 (GPIO2/ADC2_CH2)
- net SHD/SD2: now also U6.3 (IO2); no longer U6.7 (IO3)
- net SWP/SD3: now also U6.7 (IO3); no longer U6.3 (IO2)
- net UART_RX: now also U2.8 (TXD); no longer U2.9 (RXD)
- net UART_TX: now also U2.9 (RXD); no longer U2.8 (TXD)
- net BAT_ADC: now reaches U1.10 (VDET_1/GPIO34/ADC1_CH6)
- net ~{CHG}: now reaches U1.12 (32K_XP/GPIO32/ADC1_CH4)
- net AUDIO_VCC_EN: now reaches U1.24 (GPIO4/ADC2_CH0)
- net EN1: now reaches U1.25 (GPIO16)
- net EN2: now reaches U1.27 (GPIO17)
- net AUDIO_SW: now reaches U1.34 (GPIO5)
- net CH340_EN: now reaches U1.42 (GPIO21)
- net CH340_EN: now also Q2.1 (G), R40.1
- net USB_CC1: now reaches U1.5 (SENSOR_VP/GPIO36/ADC1_CH0)
- net USB_CC2: now reaches U1.6 (SENSOR_CAPP/GPIO37/ADC1_CH1)
- net ~{PGOOD}: now reaches U1.7 (SENSOR_CAPN/GPIO38/ADC1_CH2)
- net USB_VBUS_SENSE: now reaches U1.8 (SENSOR_VN/GPIO39/ADC1_CH3)
- net +3V3 renamed +3V3_SYS
- net +3V3_SYS: now also Q2.2 (S); no longer C19.1, U2.10 (V3), U2.7 (VCC)
- new net: C19.1, Q2.3 (D), U2.10 (V3), U2.7 (VCC)
- new net ~{CHARGE_EN}: U1.22 (GPIO2/ADC2_CH2)
- no-connect marks 14 -> 3
Other:
- moved on the sheet: C10, C11, C33, C7, C8, C9, J3, TP9
