File: hw/bluetooth-audio/micro.kicad_sch (KiCad schematic)
At the start: 49 parts, among them J3 Conn_01x06, J4 2x5 JTAG header, Q1 UMH3N, Q2 AO3401A, U1 ESP32D0WD-V3, U2 CH340K, U6 W25Q32JVZP, Y1 Crystal 40 MHz 10pF

Commit message: Audio sheet redesign: ZTS6216 mic, PJ-3537S jack, shared 47 uF coupling
Rework the audio subsystem and record the rationale.

- Microphone: switch to ZillTek ZTS6216 (self-biased single-ended, C0G
  mic coupling C41/C42 per datasheet); pseudo-diff RIN1 provisioned DNP.
- Jack: PJ-3537S 3-pole TRS + detect switch (custom symbol + footprint).
- Coupling: single shared 47 uF electrolytic pair (C1/C21) on the jack
  side of the TX/RX switch, serving both RX and TX; R22/R23 bleed.
- TX input: BAT54S series-Schottky clamps (D7/D8) to AVDD/GND,
  line-level-only, PGA 0 dB.
- Ground loop: battery-only playback is the plan of record (no
  transformer footprint).
- Add TS5A23159 switch, ZTS6216 and PJ-3537S datasheets.
- Add systems design review (docs/design-review-audio.md) and update
  design overview with coupling-cap sizing.
- PCB layout updated to match.

Co-Authored-By: Claude Opus 4.8 <noreply@anthropic.com>
Parts:
- removed R19, R20: 4k7, Resistor_SMD:R_0402_1005Metric, symbol Device:R_Small
Connections:
- no-connect marks 3 -> 4

Commit message: BOM sanity check: fix part numbers, populate passives, normalise fields
Full footprint + LCSC audit across power/audio/micro sheets (see
docs/bom-audit.md). Every part now carries Manufacturer + MPN + LCSC in one
consistent field set, validated against the jlcparts snapshot.

Corrections:
- Fix C1849 mis-assignment: it is a 10uF 1206 MLCC that had been pasted onto
  14 caps of unrelated values (incl. the 18pF crystal load caps); each
  reassigned to the correct part, stale Supplier Part Number cleared.
- D1 LED_BLUE was a white LED (C34499) -> C2293 (KT-0805B, blue).
- Populate all resistors/caps/L1 with JLCPCB parts (Basic where available;
  C0G for crystal-load 18pF, RF 3.3pF, and preserved on audio 100nF C41/C42).
- C48 SYS bulk MLCC -> 47uF/10V tantalum C22036 (DC-bias); footprint 3528-21.
- C27 10uF 0402 -> 0603 (match siblings). C19702.
- U3 footprint TSSOP-10 -> MSOP-10 (DGS = VSSOP, no thermal pad); C42751.
- Q2 -> C15127, J2 -> C5143397 (GCT USB-C), D6 LED_CHG -> amber C2296.
- J5 Molex -> JST-PH 3-pin battery connector S3B-PH-K-S (C157929).
- U9 (BQ24074 charger) marked DNP.
- Migrate all ICs/LEDs/discretes from Supplier Part Number to LCSC + add
  Manufacturer/MPN.

Adds docs/bom-audit.md with the priced BOM (~$11/board at 30 qty) and open
items (battery selection, U9 DNP, PCB re-sync).

Co-Authored-By: Claude Opus 4.8 <noreply@anthropic.com>
Parts:
- C10, C11, C19, C33, C9: LCSC (none) -> C1525; MPN (none) -> CL05B104KO5NNNC; Manufacturer (none) -> Samsung Electro Mechanics
- C34, C6, C7: LCSC (none) -> C52923; MPN (none) -> CL05A105KA5NQNC; Manufacturer (none) -> Samsung Electro Mechanics; Supplier Part Number C1849 -> (none)
- C35: LCSC (none) -> C1549; MPN (none) -> 0402CG180J500NT; Manufacturer (none) -> FH Guangdong Fenghua Advanced Tech; Supplier Part Number C1849 -> (none)
- C36: LCSC (none) -> C1549; MPN (none) -> 0402CG180J500NT; Manufacturer (none) -> FH Guangdong Fenghua Advanced Tech
- C37, C38: LCSC (none) -> C76906; MPN (none) -> GJM1555C1H3R3BB01D; Manufacturer (none) -> Murata Electronics
- C45: LCSC (none) -> C15195; MPN (none) -> CL05B103KB5NNNC; Manufacturer (none) -> Samsung Electro Mechanics
- C8: LCSC (none) -> C19702; MPN (none) -> CL10A106KP8NNNC; Manufacturer (none) -> Samsung Electro Mechanics; Supplier Part Number C1849 -> (none)
- D1: LCSC (none) -> C2293; MPN (none) -> KT-0805B; Manufacturer (none) -> Hubei KENTO Elec; Supplier Part Number C34499 -> (none)
- D3: LCSC (none) -> C2297; MPN (none) -> KT-0805G; Manufacturer (none) -> Hubei KENTO Elec; Supplier Part Number C2297 -> (none)
- L1: LCSC (none) -> C86061; MPN (none) -> LQG15HS2N2S02D; Manufacturer (none) -> Murata Electronics
- Q1: LCSC (none) -> C62892; MPN (none) -> UMH3N; Manufacturer (none) -> Jiangsu Changjing Electronics; Supplier Part Number C62892 -> (none)
- Q1: Supplier Part Number C62892 -> (none)
- Q2: LCSC (none) -> C15127; MPN (none) -> AO3401A; Manufacturer (none) -> Alpha Omega Semicon
- R1, R11, R2: LCSC (none) -> C25744; MPN (none) -> 0402WGF1002TCE; Manufacturer (none) -> UNI ROYAL Uniroyal Elec
- R12, R18: LCSC (none) -> C25104; MPN (none) -> 0402WGF3300TCE; Manufacturer (none) -> UNI ROYAL Uniroyal Elec
- R13, R14, R3: LCSC (none) -> C17168; MPN (none) -> 0402WGF0000TCE; Manufacturer (none) -> UNI ROYAL Uniroyal Elec
- R24, R25, R26: LCSC (none) -> C25900; MPN (none) -> 0402WGF4701TCE; Manufacturer (none) -> UNI ROYAL Uniroyal Elec
- R40: LCSC (none) -> C25741; MPN (none) -> 0402WGF1003TCE; Manufacturer (none) -> UNI ROYAL Uniroyal Elec
- U1: LCSC (none) -> C967021; MPN (none) -> ESP32-D0WD-V3; Manufacturer (none) -> Espressif Systems; Supplier Part Number C967021 -> (none)
- U2: LCSC (none) -> C968586; MPN (none) -> CH340K; Manufacturer (none) -> WCH(Jiangsu Qin Heng); Supplier Part Number C968586 -> (none)
- U6: LCSC (none) -> C571260; MPN (none) -> W25Q32JVZPIQ; Manufacturer (none) -> Winbond Elec; Supplier Part Number C571260 -> (none)
- Y1: LCSC (none) -> C255898; MPN (none) -> Q22FA12800101; Manufacturer (none) -> Seiko Epson; Supplier Part Number C255898 -> (none)

Commit message: BOM: move C51, charger resistors and D1 to JLCPCB Basic parts
Cuts Extended (paid-setup) parts from 25 to 20 without changing any circuit
values:
- C51 USB-shield filter 4.7nF: 1206 -> 0402, Basic C1538 (generic filter cap).
- R_TMR1/R_ISET1/R_ITERM1 (56k/1.2k/3k charger programming): 0402 -> 0603 to
  get Basic parts at the SAME values (C23206/C22765/C4211) - charger behaviour
  unchanged; no Basic exists at these values in 0402.
- D1: no blue LED is a JLCPCB Basic part, so changed to white (C34499, Basic);
  value relabelled LED_WHITE. GPIO net still named LED_BLUE.

Left Extended (no Basic option / intentional):
- C37/C38 are the 2.4GHz antenna-match caps (need NP0), not crystal-load caps;
  no Basic 3.3pF exists. Crystal-load caps are C35/C36 (already Basic C0G).
- Q1 UMH3N: no Basic dual/single digital transistor - see docs/bom-audit.md
  section 6 (keep Extended vs redesign to 2x MMBT3904 + resistors).

docs/bom-audit.md updated with the changes and revised cost (~$11.24/board @30).

Co-Authored-By: Claude Opus 4.8 <noreply@anthropic.com>
Parts:
- D1: value LED_BLUE -> LED_WHITE; LCSC C2293 -> C34499; MPN KT-0805B -> KT-0805W
Changed lines of the file:
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@@
 			)
 		)
-		(property "Value" "LED_BLUE"
+		(property "Value" "LED_WHITE"
 			(at 251.46 92.6465 90)
 			(show_name no)
@@
 			)
 		)
-		(property "MPN" "KT-0805B"
+		(property "MPN" "KT-0805W"
 			(at 248.92 91.44 0)
 			(hide yes)
@@
 			)
 		)
-		(property "LCSC" "C2293"
+		(property "LCSC" "C34499"
 			(at 248.92 91.44 0)
 			(hide yes)

Commit message: Audio BOM: OUT2 couplers to electrolytic, C53 0402, C41/C42 land; place PCB
Schematic (audio + power sheets):
- C24/C26 (ES8388 OUT2 -> TP6 test-output couplers): 1uF MLCC -> 47uF
  electrolytic (Panasonic EEEFT1E470AR / C336270), matching C1/C21. Polarity
  verified against the netlist: + terminal to the codec/VMID side.
- C53 (USB_VBUS_SENSE divider filter): 1206 -> 0402 (house part
  CL05B104KO5NNNC / C1525).
- C41/C42 (mic C0G couplers): footprint aligned to plain C_1206_3216Metric,
  matching C54.

PCB: all footprints now placed in their initial positions, pending V1 routing.

Docs: design-overview.tex updated (delta #20 + 2026-09-16 revision entry). The
D7/D8 TX-input clamp removal is decided but recorded as pending -- that
schematic edit is being done by hand and is not in this commit.

Note: the deleted kicad-library submodule and the untracked in-project library
copies are deliberately left unstaged (broken/redundant state).

Co-Authored-By: Claude Opus 4.8 <noreply@anthropic.com>
Parts:
- removed R1, R2: 10k, Resistor_SMD:R_0402_1005Metric, symbol Device:R_Small
- Y1: footprint Crystal:Crystal_SMD_SeikoEpson_FA128-4Pin_2.0x1.6mm -> Crystal:Crystal_SMD_2520-4Pin_2.5x2.0mm; LCSC C255898 -> C1021653; MPN Q22FA12800101 -> E2SB40E000006E; Manufacturer Seiko Epson -> Hosonic Elec
Connections:
- net DTR: now also Q1.2 (B1)
- net RTS: now also Q1.5 (B2)
- net LED_BLUE renamed LED_WHITE
