File: hw/bluetooth-audio/power.kicad_sch (KiCad schematic)
At the start: 46 parts, among them J2 USB_C_Receptacle_USB2.0, J5 Conn_01x03, U11 LP5907MFX-3.3, U5 USBLC6-2SC6, U7 AP7361C-33Y5, U9 BQ24074RGT

Commit message: Audio sheet redesign: ZTS6216 mic, PJ-3537S jack, shared 47 uF coupling
Rework the audio subsystem and record the rationale.

- Microphone: switch to ZillTek ZTS6216 (self-biased single-ended, C0G
  mic coupling C41/C42 per datasheet); pseudo-diff RIN1 provisioned DNP.
- Jack: PJ-3537S 3-pole TRS + detect switch (custom symbol + footprint).
- Coupling: single shared 47 uF electrolytic pair (C1/C21) on the jack
  side of the TX/RX switch, serving both RX and TX; R22/R23 bleed.
- TX input: BAT54S series-Schottky clamps (D7/D8) to AVDD/GND,
  line-level-only, PGA 0 dB.
- Ground loop: battery-only playback is the plan of record (no
  transformer footprint).
- Add TS5A23159 switch, ZTS6216 and PJ-3537S datasheets.
- Add systems design review (docs/design-review-audio.md) and update
  design overview with coupling-cap sizing.
- PCB layout updated to match.

Co-Authored-By: Claude Opus 4.8 <noreply@anthropic.com>
Parts:
- R39: value 47k -> 100k
- renumbered R_ILIM to R_ILIM1, R_ISET to R_ISET1, R_ITERM to R_ITERM1, R_NTC_LIN to R_NTC_LIN1, R_TMR to R_TMR1
Connections:
- net USB_VBUS_SENSE: no longer C53.1
Changed lines of the file:
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@@
 	)
 	(junction
-		(at 130.81 31.75)
-		(diameter 0)
-		(color 0 0 0 0)
-	)
-	(junction
 		(at 139.7 160.02)
 		(diameter 0)
@@
 		(in_pos_files yes)
 		(dnp no)
-		(property "Reference" "R_TMR"
+		(property "Reference" "R_TMR1"
 			(at 96.774 132.334 90)
 			(show_name no)
@@
 			(project "bluetooth-audio"
 				(path "/eafc8824-f117-40b2-99b0-597946d6c01d/541dab54-ea50-443b-9935-4ff5142dd0fa"
-					(reference "R_TMR")
+					(reference "R_TMR1")
 					(unit 1)
 				)
@@
 		(dnp yes)
 		(fields_autoplaced yes)
-		(property "Reference" "R_NTC_LIN"
+		(property "Reference" "R_NTC_LIN1"
 			(at 54.61 114.2999 0)
 			(show_name no)
@@
 			(project "bluetooth-audio"
 				(path "/eafc8824-f117-40b2-99b0-597946d6c01d/541dab54-ea50-443b-9935-4ff5142dd0fa"
-					(reference "R_NTC_LIN")
+					(reference "R_NTC_LIN1")
 					(unit 1)
 				)
@@
 			)
 		)
-		(property "Value" "47k"
+		(property "Value" "100k"
 			(at 123.19 39.878 0)
 			(show_name no)
@@
 		(dnp no)
 		(fields_autoplaced yes)
-		(property "Reference" "R_ITERM"
+		(property "Reference" "R_ITERM1"
 			(at 96.52 116.84 90)
 			(show_name no)
@@
 			(project "bluetooth-audio"
 				(path "/eafc8824-f117-40b2-99b0-597946d6c01d/541dab54-ea50-443b-9935-4ff5142dd0fa"
-					(reference "R_ITERM")
+					(reference "R_ITERM1")
 					(unit 1)
 				)
@@
 		(in_pos_files yes)
 		(dnp no)
-		(property "Reference" "R_ILIM"
+		(property "Reference" "R_ILIM1"
 			(at 97.79 167.6399 0)
 			(show_name no)
@@
 			(project "bluetooth-audio"
 				(path "/eafc8824-f117-40b2-99b0-597946d6c01d/541dab54-ea50-443b-9935-4ff5142dd0fa"
-					(reference "R_ILIM")
+					(reference "R_ILIM1")
 					(unit 1)
 				)
@@
 		(in_pos_files yes)
 		(dnp no)
-		(property "Reference" "R_ISET"
+		(property "Reference" "R_ISET1"
 			(at 106.68 167.6399 0)
 			(show_name no)
@@
 			(project "bluetooth-audio"
 				(path "/eafc8824-f117-40b2-99b0-597946d6c01d/541dab54-ea50-443b-9935-4ff5142dd0fa"
-					(reference "R_ISET")
+					(reference "R_ISET1")
 					(unit 1)
 				)

Commit message: BOM sanity check: fix part numbers, populate passives, normalise fields
Full footprint + LCSC audit across power/audio/micro sheets (see
docs/bom-audit.md). Every part now carries Manufacturer + MPN + LCSC in one
consistent field set, validated against the jlcparts snapshot.

Corrections:
- Fix C1849 mis-assignment: it is a 10uF 1206 MLCC that had been pasted onto
  14 caps of unrelated values (incl. the 18pF crystal load caps); each
  reassigned to the correct part, stale Supplier Part Number cleared.
- D1 LED_BLUE was a white LED (C34499) -> C2293 (KT-0805B, blue).
- Populate all resistors/caps/L1 with JLCPCB parts (Basic where available;
  C0G for crystal-load 18pF, RF 3.3pF, and preserved on audio 100nF C41/C42).
- C48 SYS bulk MLCC -> 47uF/10V tantalum C22036 (DC-bias); footprint 3528-21.
- C27 10uF 0402 -> 0603 (match siblings). C19702.
- U3 footprint TSSOP-10 -> MSOP-10 (DGS = VSSOP, no thermal pad); C42751.
- Q2 -> C15127, J2 -> C5143397 (GCT USB-C), D6 LED_CHG -> amber C2296.
- J5 Molex -> JST-PH 3-pin battery connector S3B-PH-K-S (C157929).
- U9 (BQ24074 charger) marked DNP.
- Migrate all ICs/LEDs/discretes from Supplier Part Number to LCSC + add
  Manufacturer/MPN.

Adds docs/bom-audit.md with the priced BOM (~$11/board at 30 qty) and open
items (battery selection, U9 DNP, PCB re-sync).

Co-Authored-By: Claude Opus 4.8 <noreply@anthropic.com>
Parts:
- removed C49: 47uF, Capacitor_SMD:C_1206_3216Metric, symbol Device:C_Small
- added C22: 4.7uF, Capacitor_SMD:C_0603_1608Metric, symbol Device:C_Small
- C2: LCSC (none) -> C1848; MPN (none) -> CL31B105KBHNNNE; Manufacturer (none) -> Samsung Electro Mechanics; Supplier Part Number C1849 -> (none)
- C20: LCSC (none) -> C15849; MPN (none) -> CL10A105KB8NNNC; Manufacturer (none) -> Samsung Electro Mechanics; Supplier Part Number C1849 -> (none)
- C3: LCSC (none) -> C29823; MPN (none) -> 1206B475K500NT; Manufacturer (none) -> FH Guangdong Fenghua Advanced Tech; Supplier Part Number C1849 -> (none)
- C4: LCSC (none) -> C19666; MPN (none) -> CL10A475KO8NNNC; Manufacturer (none) -> Samsung Electro Mechanics; Supplier Part Number C1849 -> (none)
- C47, C5, C50: LCSC (none) -> C13585; MPN (none) -> CL31A106KBHNNNE; Manufacturer (none) -> Samsung Electro Mechanics; Supplier Part Number C1849 -> (none)
- C48: footprint Capacitor_SMD:C_1206_3216Metric -> Capacitor_Tantalum_SMD:CP_EIA-3528-21_Kemet-B; LCSC (none) -> C22036; MPN (none) -> TAJB476K010RNJ; Manufacturer (none) -> Kyocera AVX; Supplier Part Number C1849 -> (none)
- C51: LCSC (none) -> C113886; MPN (none) -> CC1206JRNPO9BN472; Manufacturer (none) -> YAGEO; Supplier Part Number C1849 -> (none)
- C52, C53: LCSC (none) -> C24497; MPN (none) -> CL31B104KBCNNNC; Manufacturer (none) -> Samsung Electro Mechanics; Supplier Part Number C1849 -> (none)
- D2, D4, D5: LCSC (none) -> C2297; MPN (none) -> KT-0805G; Manufacturer (none) -> Hubei KENTO Elec; Supplier Part Number C2297 -> (none)
- D6: LCSC (none) -> C2296; MPN (none) -> KT-0805Y; Manufacturer (none) -> Hubei KENTO Elec; Supplier Part Number C2297 -> (none)
- J2: LCSC (none) -> C5143397; MPN (none) -> USB4110-GF-A; Manufacturer (none) -> Global Connector Technology
- J5: footprint Connector_Molex:Molex_Micro-Latch_53254-0370_1x03_P2.00mm_Horizontal -> Connector_JST:JST_PH_S3B-PH-K_1x03_P2.00mm_Horizontal; LCSC (none) -> C157929; MPN (none) -> S3B-PH-K-S(LF)(SN); Manufacturer (none) -> JST
- R15, R28, R29, R6: LCSC (none) -> C25104; MPN (none) -> 0402WGF3300TCE; Manufacturer (none) -> UNI ROYAL Uniroyal Elec
- R17, R30, R31, R34, R35, R38, R39: LCSC (none) -> C25741; MPN (none) -> 0402WGF1003TCE; Manufacturer (none) -> UNI ROYAL Uniroyal Elec
- R32, R33, R36, R37, R_NTC_LIN1: LCSC (none) -> C11702; MPN (none) -> 0402WGF1001TCE; Manufacturer (none) -> UNI ROYAL Uniroyal Elec
- R4, R5: LCSC (none) -> C25905; MPN (none) -> 0402WGF5101TCE; Manufacturer (none) -> UNI ROYAL Uniroyal Elec
- R_ILIM1: LCSC (none) -> C25867; MPN (none) -> 0402WGF1501TCE; Manufacturer (none) -> UNI ROYAL Uniroyal Elec
- R_ISET1: LCSC (none) -> C2909307; MPN (none) -> FRC0402F1201TS; Manufacturer (none) -> FOJAN
- R_ITERM1: LCSC (none) -> C2909355; MPN (none) -> FRC0402F3001TS; Manufacturer (none) -> FOJAN
- R_TMR1: LCSC (none) -> C2906875; MPN (none) -> FRC0402F5602TS; Manufacturer (none) -> FOJAN
- U11: LCSC (none) -> C80670; MPN (none) -> LP5907MFX-3.3/NOPB; Manufacturer (none) -> Texas Instruments
- U5: LCSC (none) -> C7519; MPN (none) -> USBLC6-2SC6; Manufacturer (none) -> STMicroelectronics; Supplier Part Number C7519 -> (none)
- U7: LCSC (none) -> C460397; MPN (none) -> AP7361C-33Y5-13; Manufacturer (none) -> Diodes Incorporated; Supplier Part Number C460397 -> (none)
- U9: LCSC (none) -> C54313; MPN (none) -> BQ24074RGTR; Manufacturer (none) -> Texas Instruments; now not fitted
Connections:
- net +BATT: now also C22.1
- net GND: now also C22.2
